File: DummyLoad.kicad_sch (KiCad schematic)
At the start: 30 parts, among them J1 YK3030423000G, J2 Conn_01x05, Q1 IRFP250N, Q2 IRFP250N, Q3 IRFP250N, U1 LM324

Commit message: Added README.md
Parts:
- removed C6: 100n, Capacitor_SMD:C_0603_1608Metric, symbol Device:C_Small
- removed J2: Conn_01x05, symbol Connector_Generic:Conn_01x05
- removed R16: 1M, Resistor_SMD:R_0603_1608Metric, symbol Device:R
- added C10, C8, C9: 1n, Capacitor_SMD:C_0603_1608Metric, symbol Device:C_Small
- added C11, C12, C13: 10n, Capacitor_SMD:C_0603_1608Metric, symbol Device:C_Small
- added C14, C15, C16, C17, C18, C21: 100n, Capacitor_SMD:C_0603_1608Metric, symbol Device:C_Small
- added C19: 2u2, Capacitor_SMD:C_0603_1608Metric, symbol Device:C_Small
- added C20: 100u, Capacitor_THT:C_Radial_D6.3mm_H7.0mm_P2.50mm, symbol Device:C_Small_US
- added D2: 1N4148, Diode_THT:D_DO-35_SOD27_P7.62mm_Horizontal, symbol Diode:1N4148
- added FB2: 220R, Inductor_SMD:L_0603_1608Metric, symbol Device:FerriteBead_Small
- added J3: Conn_01x08, symbol Connector_Generic:Conn_01x08
- added K1: G2RL-1-E, Relay_THT:Relay_SPDT_Omron_G2RL-1-E, symbol Relay:G2RL-1-E
- added Q4: 2N7002, Package_TO_SOT_SMD:SOT-23, symbol Transistor_FET:2N7002
- added R17: 0R01, Resistor_THT:R_Bare_Metal_Element_L21.3mm_W4.8mm_P20.30mm, symbol Device:R
- added R18: 0R1, Resistor_THT:R_Bare_Metal_Element_L21.3mm_W4.8mm_P20.30mm, symbol Device:R
- added R19: 4k7, Resistor_SMD:R_0603_1608Metric, symbol Device:R
- added U2: MCP3422Axx-xSN, Package_SO:SOIC-8_3.9x4.9mm_P1.27mm, symbol Analog_ADC:MCP3422Axx-xSN
- added U3, U4: INA180A1, Package_TO_SOT_SMD:SOT-23-5, symbol Amplifier_Current:INA180A1
- C7: Link (none) -> https://www.tme.eu/pl/en/details/cc-104_500/ceramic-capacit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
- R1, R10, R14, R15, R2, R3: Link (none) -> https://allegro.pl/produkt/rezystor-3w-0-1r-royal-ohm-knp-2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
Connections:
- net +15V: now also C1.1, C2.1, FB1.1, U1.4 (V+); no longer C4.1, C5.1, FB1.2
- net F0: now also C9.1
- net F1: now also C8.1
- net F2: now also C10.1
- net Masa: now also C11.2, C12.2, C13.2, C14.2, C15.2, C16.2, C17.2, C18.2, C19.2, C20.2, C21.2, J3.4 (Pin_4), J3.5 (Pin_5), J3.8 (Pin_8), Q4.2 (S), R17.2, R18.2, R19.2, U2.2 (CH1-), U2.6 (V_{SS}), U2.8 (CH2-), U3.2 (GND), U3.4 (-), U4.2 (GND), U4.4 (-); no longer R1.2, R10.2, R14.2, R15.2, R2.2, R3.2
- net at R13.2, U1.10 (+): now also C13.1
- net at R9.1, U1.8: now also C10.2
- net at R7.1, U1.1: now also C9.2
- net at R12.2, U1.3 (+): now also C11.1
- net at R8.1, U1.7: now also C8.2
- net at R11.2, U1.5 (+): now also C12.1
- new net: K1.14, R18.1, U4.3 (+)
- new net: C4.1, C5.1, FB1.2, J3.2 (Pin_2)
- new net: K1.11, R1.2, R10.2, R14.2, R15.2, R2.2, R3.2
- new net: K1.12, R17.1, U3.3 (+)
- new net: D2.2 (A), K1.A1, Q4.3 (D)
- new net: C20.1, C21.1, FB2.2, J3.3 (Pin_3)
- new net +24V: C17.1, D2.1 (K), J3.1 (Pin_1), K1.A2
- new net +5V: C14.1, C15.1, C16.1, C18.1, C19.1, FB2.1, U2.3 (V_{DD}), U3.5 (V+), U4.5 (V+)
- new net RangeSelect: Q4.1 (G), R19.1
- new net SCL: J3.7 (Pin_7), U2.5 (SCL)
- new net SDA: J3.6 (Pin_6), U2.4 (SDA)
- new net Sense0: U2.1 (CH1+), U3.1
- new net Sense1: U2.7 (CH2+), U4.1
Other:
- added sheet ControlBoard (ControlBoard.kicad_sch)
- note added: "+24V +15V +5V - Det SDA SCL"
- note added: "TODO: DAC Connector"
- note removed: "+ - Det Ref -"
- note removed: "x4"
- moved on the sheet: C1, C2, C4, C5, C7, FB1, J1, Q1, Q2, Q3, R1, R11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

Commit message: sync
Parts:
- removed C16: 100n, Capacitor_SMD:C_0603_1608Metric, symbol Device:C_Small
- removed D2: 1N4148, Diode_THT:D_DO-35_SOD27_P7.62mm_Horizontal, symbol Diode:1N4148
- removed J3: Conn_01x08, symbol Connector_Generic:Conn_01x08
- removed U2: MCP3422Axx-xSN, Package_SO:SOIC-8_3.9x4.9mm_P1.27mm, symbol Analog_ADC:MCP3422Axx-xSN
- added D2: 1N4148W, Diode_SMD:D_SOD-123, symbol Diode:1N4148W
- added J3: Conn_01x10, Connector_PinHeader_2.54mm:PinHeader_1x10_P2.54mm_Vertical, symbol Connector_Generic:Conn_01x10
Connections:
- net +24V: now also D2.1 (K), J3.1 (Pin_1)
- net Masa: now also J3.10 (Pin_10), J3.4 (Pin_4), J3.5 (Pin_5)
- net RangeSelect: now also J3.8 (Pin_8)
- net Sense0: now also J3.6 (Pin_6)
- net Sense1: now also J3.7 (Pin_7)
- net Set: now also J3.9 (Pin_9)
- net at C4.1, C5.1, FB1.2: now also J3.2 (Pin_2)
- net at K1.A1, Q4.3 (D): now also D2.2 (A)
- net at C20.1, C21.1, FB2.2: now also J3.3 (Pin_3)
Other:
- added sheet MCU (MCU.kicad_sch)
- added sheet VRM (VRM.kicad_sch)
- note added: "+24V +15V +5V - Det Sense0 Sense1 RangeSelect Set -"
- note removed: "+24V +15V +5V - Det SDA SCL"
