File: MCU.kicad_sch (KiCad schematic)
At the start: 42 parts, among them J10 Screw_Terminal_01x03, J11 Conn_01x04, J12 USB4105-GF-A-120, J8 Conn_01x14, J9 Conn_01x04, M1 Fan_4pin, M2 Fan_4pin, M3 Fan_4pin, M4 Fan_4pin, U10 TMP102xxDRL, U7 STM32G431C6Tx, U8 USBLC6-2SC6, U9 FM24C64B, Y1 Crystal_GND24

Commit message: sync
Parts:
- C39: Link https://www.mouser.pl/en/ProductDetail/Samsung-Electro-Mech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 -> (none); Price 0,36zł -> (none)
- FB3: Link https://www.mouser.pl/en/ProductDetail/TDK/MMZ1608S121ATA00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 -> (none); Price 0,36zł -> (none)
Changed lines of the file:
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@@
 			)
 		)
-		(property "Link" "https://www.mouser.pl/en/ProductDetail/Samsung-Electro-Mechanics/CL10A225KP8NNNC?qs=sGAEpiMZZMs7ZEmUmaUL039fXNp4KT2O5Ksi0Uzem1c%3D"
+		(property "Link" ""
 			(at 257.81 52.07 0)
 			(hide yes)
@@
 			)
 		)
-		(property "Price" "0,36zł "
+		(property "Price" ""
 			(at 257.81 52.07 0)
 			(hide yes)
@@
 			)
 		)
-		(property "Link" "https://www.mouser.pl/en/ProductDetail/TDK/MMZ1608S121ATA00?qs=sGAEpiMZZMt1hubY80%2Fs8EvTGpImDuNGEL%252BoYtFtc14%3D"
+		(property "Link" ""
 			(at 266.7 49.53 90)
 			(hide yes)
@@
 			)
 		)
-		(property "Price" "0,36zł "
+		(property "Price" ""
 			(at 266.7 49.53 90)
 			(hide yes)
