File: PCB/ControlBoard/ControlBoard.kicad_sch (KiCad schematic)
At the start: 117 parts, among them J1 Conn_01x05, J10 Screw_Terminal_01x03, J11 Conn_01x04, J12 USB4105-GF-A-120, J13 Screw_Terminal_01x02, J14 Screw_Terminal_01x02, J2 Conn_01x05, J4 Conn_01x10, J5 Conn_01x10, J6 Conn_01x10, J7 Conn_01x10, J8 Conn_01x14, J9 Conn_01x04, M1 Fan_4pin, M2 Fan_4pin, M3 Fan_4pin, M4 Fan_4pin, U10 TMP102xxDRL, U11 L7815, U12 MCP4728, U13 L7805, U14 SD8942, U2 ADS1115IDGS, U5 74HC4051, U6 LMR33630ADDA, U7 STM32G431C6Tx, U8 USBLC6-2SC6, U9 FM24C64B, Y1 Crystal_GND24

Commit message: Fixed MCU Reset Line
Parts:
- added C66: 100n, Capacitor_SMD:C_0603_1608Metric, symbol Device:C_Small
- added R41: 10k, Resistor_SMD:R_0603_1608Metric, symbol Device:R
Connections:
- net +3V3: now also R41.1
- net Masa: now also C66.2
- net ~{RST}: now reaches U7.7 (PG10)
- net ~{RST}: now also C66.1, R41.2
